File: pcb/tactical-tenkey.kicad_sch (KiCad schematic)
At the start: 0 parts

Commit message: schematic
Parts:
- added D1, D10, D11, D12, D13, D14, D15, D16, D2, D3, D4, D5, D6, D7, D8, D9: ~, symbol ScottoKeebs:Placeholder_Diode
- added J1: Conn_01x02_Pin, symbol Connector:Conn_01x02_Pin
- added S_*, S_+, S_-, S_., S_/, S_0, S_1, S_2, S_3, S_4, S_5, S_6, S_7, S_8, S_9, S_enter, S_num: ~, symbol ScottoKeebs:Placeholder_Keyswitch
- added U1: XIAO-ESP32-S3-SMD, Seeed_Studio_XIAO_Series:XIAO-ESP32-S3-SMD, symbol seeed_esp32:XIAO-ESP32-S3-SMD
Connections:
- new net: J1.2 (Pin_2), U1.32 (BAT)
- new net: J1.1 (Pin_1), U1.33 (GND)
- new net: D6.2 (A), S_8.2
- new net: D11.2 (A), S_1.2
- new net: D5.2 (A), S_7.2
- new net: D3.2 (A), S_*.2
- new net: D1.2 (A), S_num.2
- new net: D14.2 (A), S_..2
- new net: D7.2 (A), S_9.2
- new net: D13.2 (A), S_3.2
- new net: D8.2 (A), S_4.2
- new net: D4.2 (A), S_-.2
- new net: D16.2 (A), S_+.2
- new net: D10.2 (A), S_6.2
- new net: D9.2 (A), S_5.2
- new net: D15.2 (A), S_0.2
- new net: D2.2 (A), S_/.2
- new net: D12.2 (A), S_2.2
- new net GND: S_enter.2, U1.13 (GND)
- new net col_1: S_1.1, S_4.1, S_7.1, S_num.1, U1.11 (GPIO9_A10_D10_MOSI)
- new net col_2: S_/.1, S_2.1, S_5.1, S_8.1, U1.10 (GPIO8_A9_D9_MISO)
- new net col_3: S_*.1, S_3.1, S_6.1, S_9.1, U1.9 (GPIO7_A8_D8_SCK)
- new net col_4: S_+.1, S_-.1, S_..1, U1.8 (GPIO44_D7_RX)
- new net pwr: S_enter.1, U1.1 (GPIO1_A0_D0)
- new net row_1: D1.1 (K), D2.1 (K), D3.1 (K), D4.1 (K), U1.28 (GPIO42_MTMS)
- new net row_2: D16.1 (K), D5.1 (K), D6.1 (K), D7.1 (K), U1.3 (GPIO3_A2_D2)
- new net row_3: D10.1 (K), D14.1 (K), D8.1 (K), D9.1 (K), U1.4 (GPIO4_A3_D3)
- new net row_4: D11.1 (K), D12.1 (K), D13.1 (K), D15.1 (K), U1.7 (GPIO43_D6_TX)
- new net scl: U1.6 (GPIO6_A5_D5_SCL)
- new net sda: U1.5 (GPIO5_A4_D4_SDA)
- no-connect marks 0 -> 10

Commit message: battery protection
Parts:
- removed J1: Conn_01x02_Pin, symbol Connector:Conn_01x02_Pin
- added C1: 0.08uF, symbol Device:C_Small_US
- added Q1: FS8205A, FS8205A:SOP65P640X120-8N, symbol FS8205A:FS8205A
- added R1, R2: 220k, symbol keyboard:Placeholder_Resistor
- added R3: 100, symbol keyboard:Placeholder_Resistor
- added R4: 1k, symbol keyboard:Placeholder_Resistor
- added SW1: SW_SPST, symbol Switch:SW_SPST
- added U2: DW01A, Package_TO_SOT_SMD:SOT-23-6, symbol Battery_Management:DW01A
- renumbered S_* to S_*1, S_+ to S_+1, S_- to S_-1, S_. to S_.1, S_/ to S_/1, S_enter to S_enter1, S_num to S_num1
Connections:
- net GND: now also Q1.6, Q1.7, R4.1
- net col_4: now also S_0.1
- net row_2: now also U1.2 (GPIO2_A1_D1); no longer U1.3 (GPIO3_A2_D2)
- net prot+: now reaches U1.32 (BAT)
- net prot+: now also R3.1, SW1.2 (B)
- new net: R1.1, R2.2, U1.3 (GPIO3_A2_D2)
- new net: R4.2, U2.2 (CS)
- new net: Q1.1, Q1.8
- new net: Q1.4, U2.1 (OD)
- new net: Q1.5, U2.3 (OC)
- new net: C1.1, R3.2, U2.5 (VCC)
- new net +BATT: R1.2, SW1.1 (A)
- new net -BATT: C1.2, Q1.2, Q1.3, R2.1, U2.6 (GND)
- no-connect marks 10 -> 12

Commit message: pcb layout
Parts:
- added J1: io_side, Connector_PinHeader_2.54mm:PinHeader_1x03_P2.54mm_Vertical, symbol Connector:Conn_01x03_Pin
- added J2: esp32_side, Connector_PinHeader_2.54mm:PinHeader_1x03_P2.54mm_Vertical, symbol Connector:Conn_01x03_Pin
- added J3: OLED, Connector_PinHeader_2.54mm:PinHeader_1x04_P2.54mm_Vertical, symbol Connector:Conn_01x04_Pin
- C1: footprint (none) -> Capacitor_THT:CP_Radial_Tantal_D4.5mm_P5.00mm
- D1, D10, D11, D12, D13, D14, D15, D16, D2, D3, D4, D5, D6, D7, D8, D9: footprint (none) -> ScottoKeebs_Components:Diode_DO-35
- R1, R2, R3, R4: footprint (none) -> Resistor_THT:R_Axial_DIN0207_L6.3mm_D2.5mm_P10.16mm_Horizontal
- SW1: footprint (none) -> Button_Switch_THT:SW_SPST_Omron_B3F-315x_Angled
- S_*1, S_-1, S_.1, S_/1, S_1, S_2, S_3, S_4, S_5, S_6, S_7, S_8, S_9: footprint (none) -> ScottoKeebs_MX:MX_PCB_1.00u
- S_+1, S_enter1: footprint (none) -> ScottoKeebs_MX:MX_PCB_2.00u_90deg
- S_0: footprint (none) -> ScottoKeebs_MX:MX_PCB_2.00u
- S_num1: footprint (none) -> ScottoKeebs_MX:MX_PCB
- U1: footprint Seeed_Studio_XIAO_Series:XIAO-ESP32-S3-SMD -> xiao:XIAO-ESP32-S3-SMD_PAD
Connections:
- net GND: now also J3.4 (Pin_4)
- net pwr: now also J1.3 (Pin_3); no longer U1.1 (GPIO1_A0_D0)
- net row_1: now also J1.1 (Pin_1); no longer U1.28 (GPIO42_MTMS)
- net at U1.12 (3V3): now also J3.3 (Pin_3)
- net at R1.1, R2.2: now also J1.2 (Pin_2); no longer U1.3 (GPIO3_A2_D2)
- net scl: no longer names the net of U1.6 (GPIO6_A5_D5_SCL)
- net scl: now also J3.2 (Pin_2)
- net sda: no longer names the net of U1.5 (GPIO5_A4_D4_SDA)
- net sda: now also J3.1 (Pin_1)
- new net: J2.3 (Pin_3), U1.1 (GPIO1_A0_D0)
- new net: J2.1 (Pin_1), U1.28 (GPIO42_MTMS)
- new net: J2.2 (Pin_2), U1.3 (GPIO3_A2_D2)
- no-connect marks 12 -> 11
Other:
- moved on the sheet: C1, Q1, R1, R2, R3, R4, SW1, U2

Commit message: routing
Parts:
- removed R1, R2: 220k, Resistor_THT:R_Axial_DIN0207_L6.3mm_D2.5mm_P10.16mm_Horizontal, symbol keyboard:Placeholder_Resistor
- removed R3: 100, Resistor_THT:R_Axial_DIN0207_L6.3mm_D2.5mm_P10.16mm_Horizontal, symbol keyboard:Placeholder_Resistor
- removed R4: 1k, Resistor_THT:R_Axial_DIN0207_L6.3mm_D2.5mm_P10.16mm_Horizontal, symbol keyboard:Placeholder_Resistor
- removed U1: XIAO-ESP32-S3-SMD, xiao:XIAO-ESP32-S3-SMD_PAD, symbol seeed_esp32:XIAO-ESP32-S3-SMD
- added BT1: 18650, Connector_PinHeader_2.54mm:PinHeader_1x02_P2.54mm_Vertical, symbol Device:Battery_Cell
- added R1, R2: 220k, Resistor_THT:R_Axial_DIN0207_L6.3mm_D2.5mm_P10.16mm_Horizontal, symbol Device:R
- added R3: 100, Resistor_THT:R_Axial_DIN0207_L6.3mm_D2.5mm_P10.16mm_Horizontal, symbol Device:R
- added R4: 1k, Resistor_THT:R_Axial_DIN0207_L6.3mm_D2.5mm_P10.16mm_Horizontal, symbol Device:R
- added U1: XIAO-ESP32-S3-SMD, Seeed_Studio_XIAO_Series:XIAO-ESP32-S3-SMD_PAD, symbol Seeed_Studio_XIAO_Series:XIAO-ESP32-S3-SMD
- S_*1, S_-1, S_.1, S_/1, S_1, S_2, S_3, S_4, S_5, S_6, S_7, S_8, S_9: footprint ScottoKeebs_MX:MX_PCB_1.00u -> ScottoKeebs_Hotswap:Hotswap_MX_Plated_1.00u
- S_+1, S_enter1: footprint ScottoKeebs_MX:MX_PCB_2.00u_90deg -> ScottoKeebs_Hotswap:Hotswap_MX_Plated_2.00u_90deg
- S_0: footprint ScottoKeebs_MX:MX_PCB_2.00u -> ScottoKeebs_Hotswap:Hotswap_MX_Plated_2.00u
- S_num1: footprint ScottoKeebs_MX:MX_PCB -> ScottoKeebs_Hotswap:Hotswap_MX_Plated_1.00u
Connections:
- net +BATT: now also BT1.1 (+)
- net -BATT: now also BT1.2 (-)
- net GND: now also R2.2, R4.2, U1.13 (GND)
- net col_1: now also U1.11 (GPIO9_A10_D10_MOSI)
- net col_2: now also U1.10 (GPIO8_A9_D9_MISO)
- net col_3: now also U1.9 (GPIO7_A8_D8_SCK)
- net col_4: now also U1.8 (GPIO44_D7_RX)
- net prot+: now also R1.1, R3.1, U1.15 (BAT)
- net pwr: now also J2.3 (Pin_3), U1.1 (GPIO1_A0_D0)
- net row_1: now also J2.1 (Pin_1), U1.21 (GPIO42_MTMS)
- net row_2: now also U1.2 (GPIO2_A1_D1)
- net row_3: now also U1.4 (GPIO4_A3_D3)
- net row_4: now also U1.7 (GPIO43_D6_TX)
- net at J3.3 (Pin_3): now also U1.12 (3V3)
- net at J2.2 (Pin_2): now also J1.2 (Pin_2), R1.2, R2.1, U1.3 (GPIO3_A2_D2)
- net at J3.1 (Pin_1): now also U1.5 (GPIO5_A4_D4_SDA)
- net at J3.2 (Pin_2): now also U1.6 (GPIO6_A5_D5_SCL)
- net at U2.2 (CS): now also R4.1
- net at C1.1, U2.5 (VCC): now also R3.2

Commit message: case
Parts:
- removed SW1: SW_SPST, Button_Switch_THT:SW_SPST_Omron_B3F-315x_Angled, symbol Switch:SW_SPST
- added SW1: SW_SPDT, Personal:SS-12F23G5, symbol Switch:SW_SPDT
- U1: footprint Seeed_Studio_XIAO_Series:XIAO-ESP32-S3-SMD_PAD -> xiao:XIAO-ESP32-S3-SMD_PAD
Connections:
- net +BATT: now also SW1.2 (B)
- net prot+: now also SW1.1 (A)
- no-connect marks 11 -> 12
Changed lines of the file:
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@@
 	)
 	(junction
-		(at 93.98 146.05)
-		(diameter 0)
-		(color 0 0 0 0)
-	)
-	(junction
 		(at 101.6 146.05)
 		(diameter 0)
@@
 		(color 0 0 0 0)
 	)
+	(junction
+		(at 93.98 143.51)
+		(diameter 0)
+		(color 0 0 0 0)
+	)
 	(no_connect
 		(at 184.15 60.96)
 	)
 	(no_connect
+		(at 93.98 148.59)
+	)
+	(no_connect
 		(at 195.58 60.96)
 	)
@@
 	(wire
 		(pts
-			(xy 93.98 140.97) (xy 93.98 146.05)
+			(xy 93.98 140.97) (xy 93.98 143.51)
 		)
 		(stroke
@@
 		)
 	)
+	(wire
+		(pts
+			(xy 93.98 143.51) (xy 93.98 146.05)
+		)
+		(stroke
+			(width 0)
+			(type default)
+		)
+	)
 	(global_label "pwr"
 		(shape input)
@@
 	)
 	(symbol
+		(lib_id "Switch:SW_SPDT")
+		(at 88.9 146.05 0)
+		(unit 1)
+		(exclude_from_sim no)
+		(in_bom yes)
+		(on_board yes)
+		(dnp no)
+		(fields_autoplaced yes)
+		(property "Reference" "SW1"
+			(at 88.9 137.16 0)
+			(effects
+				(font
+					(size 1.27 1.27)
+				)
+			)
+		)
+		(property "Value" "SW_SPDT"
+			(at 88.9 139.7 0)
+			(effects
+				(font
+					(size 1.27 1.27)
+				)
+			)
+		)
+		(property "Footprint" "Personal:SS-12F23G5"
+			(at 88.9 146.05 0)
+			(effects
+				(font
+					(size 1.27 1.27)
+				)
+				(hide yes)
+			)
+		)
+		(property "Datasheet" "~"
+			(at 88.9 153.67 0)
+			(effects
+				(font
+					(size 1.27 1.27)
+				)
+				(hide yes)
+			)
+		)
+		(property "Description" "Switch, single pole double throw"
+			(at 88.9 146.05 0)
+			(effects
+				(font
+					(size 1.27 1.27)
+				)
+				(hide yes)
+			)
+		)
+		(pin "3"
+		)
+		(pin "2"
+		)
+		(pin "1"
+		)
+		(instances
+			(project ""
+				(path "/0d362948-d01f-4080-aaa1-0ac3b9a8002f"
+					(reference "SW1")
+					(unit 1)
+				)
+			)
+		)
+	)
+	(symbol
 		(lib_id "ScottoKeebs:Placeholder_Keyswitch")
 		(at 107.95 76.2 0)
@@
 			)
 		)
-		(property "Footprint" "Seeed_Studio_XIAO_Series:XIAO-ESP32-S3-SMD_PAD"
+		(property "Footprint" "xiao:XIAO-ESP32-S3-SMD_PAD"
 			(at 176.53 78.74 0)
 			(effects
@@
 					(unit 1)
 				)
-			)
-		)
-	)
-	(symbol
-		(lib_id "Switch:SW_SPST")
-		(at 88.9 146.05 0)
-		(unit 1)
-		(exclude_from_sim no)
-		(in_bom yes)
-		(on_board yes)
-		(dnp no)
-		(fields_autoplaced yes)
-		(property "Reference" "SW1"
-			(at 88.9 139.7 0)
-			(effects
-				(font
-					(size 1.27 1.27)
-				)
-			)
-		)
-		(property "Value" "SW_SPST"
-			(at 88.9 142.24 0)
-			(effects
-				(font
-					(size 1.27 1.27)
-				)
-			)
-		)
-		(property "Footprint" "Button_Switch_THT:SW_SPST_Omron_B3F-315x_Angled"
-			(at 88.9 146.05 0)
-			(effects
-				(font
-					(size 1.27 1.27)
-				)
-				(hide yes)
-			)
-		)
-		(property "Datasheet" "~"
-			(at 88.9 146.05 0)
-			(effects
-				(font
-					(size 1.27 1.27)
-				)
-				(hide yes)
-			)
-		)
-		(property "Description" "Single Pole Single Throw (SPST) switch"
-			(at 88.9 146.05 0)
-			(effects
-				(font
-					(size 1.27 1.27)
-				)
-				(hide yes)
-			)
-		)
-		(pin "1"
-		)
-		(pin "2"
-		)
-		(instances
-			(project ""
-				(path "/0d362948-d01f-4080-aaa1-0ac3b9a8002f"
-					(reference "SW1")
-					(unit 1)
-				)

Commit message: case development
Parts:
- S_+1, S_enter1: footprint ScottoKeebs_Hotswap:Hotswap_MX_Plated_2.00u_90deg -> ScottoKeebs_Hotswap:Hotswap_MX_Plated_2.00u
Changed lines of the file:
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@@
 			)
 		)
-		(property "Footprint" "ScottoKeebs_Hotswap:Hotswap_MX_Plated_2.00u_90deg"
+		(property "Footprint" "ScottoKeebs_Hotswap:Hotswap_MX_Plated_2.00u"
 			(at 124.46 107.95 0)
 			(effects
@@
 			)
 		)
-		(property "Footprint" "ScottoKeebs_Hotswap:Hotswap_MX_Plated_2.00u_90deg"
+		(property "Footprint" "ScottoKeebs_Hotswap:Hotswap_MX_Plated_2.00u"
 			(at 120.65 82.55 0)
 			(effects

Commit message: art
Parts:
- U1: footprint xiao:XIAO-ESP32-S3-SMD_PAD -> Seeed_Studio_XIAO_Series:XIAO-ESP32-S3-SMD_PAD
Changed lines of the file:
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@@
 			)
 		)
-		(property "Footprint" "xiao:XIAO-ESP32-S3-SMD_PAD"
+		(property "Footprint" "Seeed_Studio_XIAO_Series:XIAO-ESP32-S3-SMD_PAD"
 			(at 176.53 78.74 0)
 			(effects

Commit message: fs8205
Parts:
- removed Q1: FS8205A, FS8205A:SOP65P640X120-8N, symbol FS8205A:FS8205A
- added Q2: FS8205, FS8205:SOT95P280X145-6N, symbol FS8205:FS8205
Connections:
- net -BATT: now also Q2.1
- net GND: now also Q2.3
- net at U2.1 (OD): now also Q2.6
- net at U2.3 (OC): now also Q2.4
- new net: Q2.2, Q2.5
Changed lines of the file:
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@@
 	)
 	(no_connect
-		(at 114.3 170.18)
+		(at 114.3 160.02)
 	)
 	(no_connect
@@
 	(wire
 		(pts
-			(xy 116.84 160.02) (xy 114.3 160.02)
-		)
-		(stroke
-			(width 0)
-			(type default)
-		)
-	)
-	(wire
-		(pts
 			(xy 104.14 165.1) (xy 101.6 165.1)
 		)
@@
 	(wire
 		(pts
+			(xy 114.3 156.21) (xy 119.38 156.21)
+		)
+		(stroke
+			(width 0)
+			(type default)
+		)
+	)
+	(wire
+		(pts
 			(xy 187.96 59.69) (xy 187.96 60.96)
 		)
@@
 	(wire
 		(pts
-			(xy 106.68 160.02) (xy 109.22 160.02)
-		)
-		(stroke
-			(width 0)
-			(type default)
-		)
-	)
-	(wire
-		(pts
 			(xy 179.07 144.78) (xy 177.8 144.78)
 		)
@@
 	(wire
 		(pts
-			(xy 114.3 160.02) (xy 114.3 156.21)
-		)
-		(stroke
-			(width 0)
-			(type default)
-		)
-	)
-	(wire
-		(pts
 			(xy 124.46 165.1) (xy 124.46 168.91)
 		)
@@
 	(wire
 		(pts
+			(xy 119.38 156.21) (xy 119.38 160.02)
+		)
+		(stroke
+			(width 0)
+			(type default)
+		)
+	)
+	(wire
+		(pts
 			(xy 92.71 86.36) (xy 92.71 99.06)
 		)
@@
 	)
 	(symbol
-		(lib_id "FS8205A:FS8205A")
-		(at 114.3 165.1 270)
-		(unit 1)
-		(exclude_from_sim no)
-		(in_bom yes)
-		(on_board yes)
-		(dnp no)
-		(fields_autoplaced yes)
-		(property "Reference" "Q1"
-			(at 117.0687 170.18 90)
-			(effects
-				(font
-					(size 1.27 1.27)
-				)
-				(justify left)
-			)
-		)
-		(property "Value" "FS8205A"
-			(at 117.0687 172.72 90)
-			(effects
-				(font
-					(size 1.27 1.27)
-				)
-				(justify left)
-			)
-		)
-		(property "Footprint" "FS8205A:SOP65P640X120-8N"
-			(at 114.3 165.1 0)
-			(effects
-				(font
-					(size 1.27 1.27)
-				)
-				(justify bottom)
-				(hide yes)
-			)
-		)
-		(property "Datasheet" ""
-			(at 114.3 165.1 0)
-			(effects
-				(font
-					(size 1.27 1.27)
-				)
-				(hide yes)
-			)
-		)
-		(property "Description" ""
-			(at 114.3 165.1 0)
-			(effects
-				(font
-					(size 1.27 1.27)
-				)
-				(hide yes)
-			)
-		)
-		(property "MF" "Fortune Semiconductor"
-			(at 114.3 165.1 0)
-			(effects
-				(font
-					(size 1.27 1.27)
-				)
-				(justify bottom)
-				(hide yes)
-			)
-		)
-		(property "MAXIMUM_PACKAGE_HEIGHT" "1.2mm"
-			(at 114.3 165.1 0)
-			(effects
-				(font
-					(size 1.27 1.27)
-				)
-				(justify bottom)
-				(hide yes)
-			)
-		)
-		(property "Package" "Package"
-			(at 114.3 165.1 0)
-			(effects
-				(font
-					(size 1.27 1.27)
-				)
-				(justify bottom)
-				(hide yes)
-			)
-		)
-		(property "Price" "None"
-			(at 114.3 165.1 0)
-			(effects
-				(font
-					(size 1.27 1.27)
-				)
-				(justify bottom)
-				(hide yes)
-			)
-		)
-		(property "Check_prices" "https://www.snapeda.com/parts/FS8205A/Fortune+Semiconductor/view-part/?ref=eda"
-			(at 114.3 165.1 0)
-			(effects
-				(font
-					(size 1.27 1.27)
-				)
-				(justify bottom)
-				(hide yes)
-			)
-		)
-		(property "STANDARD" "IPC 7351B"
-			(at 114.3 165.1 0)
-			(effects
-				(font
-					(size 1.27 1.27)
-				)
-				(justify bottom)
-				(hide yes)
-			)
-		)
-		(property "PARTREV" "1.7"
-			(at 114.3 165.1 0)
-			(effects
-				(font
-					(size 1.27 1.27)
-				)
-				(justify bottom)
-				(hide yes)
-			)
-		)
-		(property "SnapEDA_Link" "https://www.snapeda.com/parts/FS8205A/Fortune+Semiconductor/view-part/?ref=snap"
-			(at 114.3 165.1 0)
-			(effects
-				(font
-					(size 1.27 1.27)
-				)
-				(justify bottom)
-				(hide yes)
-			)
-		)
-		(property "MP" "FS8205A"
-			(at 114.3 165.1 0)
-			(effects
-				(font
-					(size 1.27 1.27)
-				)
-				(justify bottom)
-				(hide yes)
-			)
-		)
-		(property "Description_1" ""
-			(at 114.3 165.1 0)
-			(effects
-				(font
-					(size 1.27 1.27)
-				)
-				(justify bottom)
-				(hide yes)
-			)
-		)
-		(property "Availability" "In Stock"
-			(at 114.3 165.1 0)
-			(effects
-				(font
-					(size 1.27 1.27)
-				)
-				(justify bottom)
-				(hide yes)
-			)
-		)
-		(property "MANUFACTURER" "Fortune Semiconductor"
-			(at 114.3 165.1 0)
-			(effects
-				(font
-					(size 1.27 1.27)
-				)
-				(justify bottom)
-				(hide yes)
-			)
-		)
-		(pin "1"
-		)
-		(pin "3"
-		)
-		(pin "8"
-		)
-		(pin "5"
-		)
-		(pin "7"
-		)
-		(pin "6"
-		)
-		(pin "4"
-		)
-		(pin "2"
-		)
-		(instances
-			(project ""
-				(path "/0d362948-d01f-4080-aaa1-0ac3b9a8002f"
-					(reference "Q1")
-					(unit 1)
-				)
-			)
-		)
-	)
-	(symbol
 		(lib_id "ScottoKeebs:Placeholder_Keyswitch")
 		(at 124.46 107.95 0)
@@
 					(unit 1)
 				)
+			)
+		)
+	)
+	(symbol
+		(lib_id "FS8205:FS8205")
+		(at 114.3 165.1 270)
+		(unit 1)
+		(exclude_from_sim no)
+		(in_bom yes)
+		(on_board yes)
+		(dnp no)
+		(property "Reference" "Q2"
+			(at 114.3 168.91 90)
+			(effects
+				(font
+					(size 1.27 1.27)
+				)
+			)
+		)
+		(property "Value" "FS8205"
+			(at 114.3 171.45 90)
+			(effects
+				(font
+					(size 1.27 1.27)
+				)
+			)
+		)
+		(property "Footprint" "FS8205:SOT95P280X145-6N"
+			(at 114.3 165.1 0)
+			(effects
+				(font
+					(size 1.27 1.27)
+				)
+				(justify bottom)
+				(hide yes)
+			)
+		)
+		(property "Datasheet" ""
+			(at 114.3 165.1 0)
+			(effects
+				(font
+					(size 1.27 1.27)
+				)
+				(hide yes)
+			)
+		)
+		(property "Description" ""
+			(at 114.3 165.1 0)
+			(effects
+				(font
+					(size 1.27 1.27)
+				)
+				(hide yes)
+			)
+		)
+		(property "MF" "Fortune Semiconductor"
+			(at 114.3 165.1 0)
+			(effects
+				(font
+					(size 1.27 1.27)
+				)
+				(justify bottom)
+				(hide yes)
+			)
+		)
+		(property "MAXIMUM_PACKAGE_HEIGHT" "1.45mm"
+			(at 114.3 165.1 0)
+			(effects
+				(font
+					(size 1.27 1.27)
+				)
+				(justify bottom)
+				(hide yes)
+			)
+		)
+		(property "Package" "Package"
+			(at 114.3 165.1 0)
+			(effects
+				(font
+					(size 1.27 1.27)
+				)
+				(justify bottom)
+				(hide yes)
+			)
+		)
+		(property "Price" "None"
+			(at 114.3 165.1 0)
+			(effects
+				(font
+					(size 1.27 1.27)
+				)
+				(justify bottom)
+				(hide yes)
+			)
+		)
+		(property "Check_prices" "https://www.snapeda.com/parts/FS8205/Fortune+Semiconductor/view-part/?ref=eda"
+			(at 114.3 165.1 0)
+			(effects
+				(font
+					(size 1.27 1.27)
+				)
+				(justify bottom)
+				(hide yes)
+			)
+		)
+		(property "STANDARD" "IPC-7351B"
+			(at 114.3 165.1 0)
+			(effects
+				(font
+					(size 1.27 1.27)
+				)
+				(justify bottom)
+				(hide yes)
+			)
+		)
+		(property "PARTREV" "1.9"
+			(at 114.3 165.1 0)
+			(effects
+				(font
+					(size 1.27 1.27)
+				)
+				(justify bottom)
+				(hide yes)
+			)
+		)
+		(property "SnapEDA_Link" "https://www.snapeda.com/parts/FS8205/Fortune+Semiconductor/view-part/?ref=snap"
+			(at 114.3 165.1 0)
+			(effects
+				(font
+					(size 1.27 1.27)
+				)
+				(justify bottom)
+				(hide yes)
+			)
+		)
+		(property "MP" "FS8205"
+			(at 114.3 165.1 0)
+			(effects
+				(font
+					(size 1.27 1.27)
+				)
+				(justify bottom)
+				(hide yes)
+			)
+		)
+		(property "Description_1" "Dual N-Channel Enhancement Mode Power MOSFET"
+			(at 114.3 165.1 0)
+			(effects
+				(font
+					(size 1.27 1.27)
+				)
+				(justify bottom)
+				(hide yes)
+			)
+		)
+		(property "Availability" "In Stock"
+			(at 114.3 165.1 0)
+			(effects
+				(font
+					(size 1.27 1.27)
+				)
+				(justify bottom)
+				(hide yes)
+			)
+		)
+		(property "MANUFACTURER" "Fortune"
+			(at 114.3 165.1 0)
+			(effects
+				(font
+					(size 1.27 1.27)
+				)
+				(justify bottom)
+				(hide yes)
+			)
+		)
+		(pin "5"
+		)
+		(pin "2"
+		)
+		(pin "1"
+		)
+		(pin "6"
+		)
+		(pin "3"
+		)
+		(pin "4"
+		)
+		(instances
+			(project ""
+				(path "/0d362948-d01f-4080-aaa1-0ac3b9a8002f"
+					(reference "Q2")
+					(unit 1)
+				)
