File: pcb/tactical-tenkey.kicad_pcb (KiCad board)
At the start: 2 copper layers, 2 parts, among them Q1 FS8205A, U2 DW01A

Commit message: pcb layout
Parts:
- added C1: 0.08uF, Capacitor_THT:CP_Radial_Tantal_D4.5mm_P5.00mm, F.Cu at (123.5, 53.5)
- added D1: ~, ScottoKeebs_Components:Diode_DO-35, F.Cu at (75.7, 65.0)
- added D10: ~, ScottoKeebs_Components:Diode_DO-35, F.Cu at (115.0, 105.5)
- added D11: ~, ScottoKeebs_Components:Diode_DO-35, F.Cu at (75.2, 125.5)
- added D12: ~, ScottoKeebs_Components:Diode_DO-35, F.Cu at (94.2, 125.5)
- added D13: ~, ScottoKeebs_Components:Diode_DO-35, F.Cu at (115.0, 125.5)
- added D14: ~, ScottoKeebs_Components:Diode_DO-35, F.Cu at (115.2, 145.0)
- added D15: ~, ScottoKeebs_Components:Diode_DO-35, F.Cu at (85.2, 145.0)
- added D16: ~, ScottoKeebs_Components:Diode_DO-35, F.Cu at (134.7, 85.0)
- added D2: ~, ScottoKeebs_Components:Diode_DO-35, F.Cu at (94.2, 65.0)
- added D3: ~, ScottoKeebs_Components:Diode_DO-35, F.Cu at (114.2, 65.0)
- added D4: ~, ScottoKeebs_Components:Diode_DO-35, F.Cu at (135.0, 65.0)
- added D5: ~, ScottoKeebs_Components:Diode_DO-35, F.Cu at (74.7, 85.5)
- added D6: ~, ScottoKeebs_Components:Diode_DO-35, F.Cu at (95.5, 85.5)
- added D7: ~, ScottoKeebs_Components:Diode_DO-35, F.Cu at (114.2, 85.5)
- added D8: ~, ScottoKeebs_Components:Diode_DO-35, F.Cu at (75.0, 105.5)
- added D9: ~, ScottoKeebs_Components:Diode_DO-35, F.Cu at (95.5, 105.5)
- added J1: io_side, Connector_PinHeader_2.54mm:PinHeader_1x03_P2.54mm_Vertical, F.Cu at (106.0, 45.5)
- added J2: esp32_side, Connector_PinHeader_2.54mm:PinHeader_1x03_P2.54mm_Vertical, F.Cu at (106.0, 50.5)
- added J3: OLED, Connector_PinHeader_2.54mm:PinHeader_1x04_P2.54mm_Vertical, F.Cu at (103.2, 59.5)
- added R1: 220k, Resistor_THT:R_Axial_DIN0207_L6.3mm_D2.5mm_P10.16mm_Horizontal, F.Cu at (104.0, 38.0)
- added R2: 220k, Resistor_THT:R_Axial_DIN0207_L6.3mm_D2.5mm_P10.16mm_Horizontal, F.Cu at (104.0, 41.5)
- added R3: 100, Resistor_THT:R_Axial_DIN0207_L6.3mm_D2.5mm_P10.16mm_Horizontal, F.Cu at (128.0, 47.0)
- added R4: 1k, Resistor_THT:R_Axial_DIN0207_L6.3mm_D2.5mm_P10.16mm_Horizontal, F.Cu at (124.5, 47.1)
- added SW1: SW_SPST, Button_Switch_THT:SW_SPST_Omron_B3F-315x_Angled, F.Cu at (73.6, 47.8)
- added S_*1: ~, ScottoKeebs_MX:MX_PCB_1.00u, F.Cu at (118.4, 75.0)
- added S_+1: ~, ScottoKeebs_MX:MX_PCB_2.00u_90deg, F.Cu at (139.3, 105.5)
- added S_-1: ~, ScottoKeebs_MX:MX_PCB_1.00u, F.Cu at (138.8, 75.0)
- added S_.1: ~, ScottoKeebs_MX:MX_PCB_1.00u, F.Cu at (118.9, 155.0)
- added S_/1: ~, ScottoKeebs_MX:MX_PCB_1.00u, F.Cu at (98.9, 74.9)
- added S_0: ~, ScottoKeebs_MX:MX_PCB_2.00u, F.Cu at (88.9, 154.9)
- added S_1: ~, ScottoKeebs_MX:MX_PCB_1.00u, F.Cu at (79.0, 135.4)
- added S_2: ~, ScottoKeebs_MX:MX_PCB_1.00u, F.Cu at (98.9, 135.5)
- added S_3: ~, ScottoKeebs_MX:MX_PCB_1.00u, F.Cu at (119.0, 135.4)
- added S_4: ~, ScottoKeebs_MX:MX_PCB_1.00u, F.Cu at (79.0, 115.4)
- added S_5: ~, ScottoKeebs_MX:MX_PCB_1.00u, F.Cu at (98.9, 115.5)
- added S_6: ~, ScottoKeebs_MX:MX_PCB_1.00u, F.Cu at (118.8, 115.5)
- added S_7: ~, ScottoKeebs_MX:MX_PCB_1.00u, F.Cu at (78.9, 95.4)
- added S_8: ~, ScottoKeebs_MX:MX_PCB_1.00u, F.Cu at (98.9, 95.5)
- added S_9: ~, ScottoKeebs_MX:MX_PCB_1.00u, F.Cu at (118.8, 95.5)
- added S_enter1: ~, ScottoKeebs_MX:MX_PCB_2.00u_90deg, F.Cu at (139.3, 145.0)
- added S_num1: ~, ScottoKeebs_MX:MX_PCB, F.Cu at (79.5, 74.9)
- added U1: XIAO-ESP32-S3-SMD, xiao:XIAO-ESP32-S3-SMD_PAD, F.Cu at (82.5, 56.0)
- moved U2 51.3 mm to (119.0, 42.0), turned to 90 degrees
- moved Q1 39.3 mm to (118.5, 50.6), turned to 90 degrees

Commit message: routing
Parts:
- added BT1: 18650, Connector_PinHeader_2.54mm:PinHeader_1x02_P2.54mm_Vertical, F.Cu at (141.4, 55.9)
- S_*1, S_-1, S_.1, S_/1, S_1, S_2, S_3, S_4, S_5, S_6, S_7, S_8, S_9: footprint ScottoKeebs_MX:MX_PCB_1.00u -> ScottoKeebs_Hotswap:Hotswap_MX_Plated_1.00u
- S_+1, S_enter1: footprint ScottoKeebs_MX:MX_PCB_2.00u_90deg -> ScottoKeebs_Hotswap:Hotswap_MX_Plated_2.00u_90deg
- S_0: footprint ScottoKeebs_MX:MX_PCB_2.00u -> ScottoKeebs_Hotswap:Hotswap_MX_Plated_2.00u
- S_num1: footprint ScottoKeebs_MX:MX_PCB -> ScottoKeebs_Hotswap:Hotswap_MX_Plated_1.00u
- U1: footprint xiao:XIAO-ESP32-S3-SMD_PAD -> Seeed_Studio_XIAO_Series:XIAO-ESP32-S3-SMD_PAD
- moved R1 28.1 mm to (127.4, 53.5), turned to 180 degrees
- moved R2 21.4 mm to (117.2, 58.3)
- moved C1 18.2 mm to (139.0, 44.0)
- moved Q1 16.6 mm to (134.2, 55.9)
- moved U2 14.2 mm to (133.1, 44.0), turned to 0 degrees
- moved SW1 12.9 mm to (72.3, 60.6)
- moved R3 11.2 mm to (117.2, 44.0), turned to 0 degrees
- moved J2 7.65 mm to (105.9, 42.9), turned to 0 degrees
- moved J1 5.15 mm to (110.4, 42.9), turned to 0 degrees
- moved U1 4.55 mm to (80.9, 60.3)
- moved S_enter1 4.29 mm to (136.6, 141.6)
- moved D14 4.16 mm to (112.8, 141.6)
- moved S_.1 4.11 mm to (117.6, 151.1)
- moved S_0 3.80 mm to (89.0, 151.1)
- moved D13 3.69 mm to (112.8, 122.5)
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Connections:
- J2 pad 1: Net-(J2-Pin_1) -> row_1
- J2 pad 2: Net-(J2-Pin_2) -> Net-(J1-Pin_2)
- J2 pad 3: Net-(J2-Pin_3) -> pwr
- R1 pad 1: Net-(J1-Pin_2) -> prot+
- R1 pad 2: +BATT -> Net-(J1-Pin_2)
- R2 pad 1: -BATT -> Net-(J1-Pin_2)
- R2 pad 2: Net-(J1-Pin_2) -> GND
- R4 pad 1: GND -> Net-(U2-CS)
- R4 pad 2: Net-(U2-CS) -> GND
- U1 pad 1: Net-(J2-Pin_3) -> pwr
- U1 pad 15: (no net) -> prot+
- U1 pad 16: (no net) -> unconnected-(U1-GND-Pad16)
- U1 pad 17: (no net) -> unconnected-(U1-GPIO41_MTDI-Pad17)
- U1 pad 18: (no net) -> unconnected-(U1-GPIO40_MTDO-Pad18)
- U1 pad 19: (no net) -> unconnected-(U1-CHIP_EN-Pad19)
- U1 pad 20: (no net) -> unconnected-(U1-GND-Pad20)
- U1 pad 21: (no net) -> row_1
- U1 pad 22: (no net) -> unconnected-(U1-GPIO39_MTCK-Pad22)
- U1 pad 23: (no net) -> unconnected-(U1-GPIO19_USB_DN-Pad23)
- U1 pad 3: Net-(J2-Pin_2) -> Net-(J1-Pin_2)
Routing:
- net row_3: track 0.00 -> 105.1 mm
- net row_1: track 0.00 -> 64.4 mm
- net row_2: track 0.00 -> 59.9 mm
- net Net-(D16-A): track 0.00 -> 14.1 mm
- net Net-(D8-A): track 0.00 -> 4.70 mm
- net Net-(D7-A): track 0.00 -> 4.58 mm
- net Net-(D6-A): track 0.00 -> 4.58 mm
- net Net-(D3-A): track 0.00 -> 4.58 mm
- net Net-(D2-A): track 0.00 -> 4.58 mm
- net Net-(D5-A): track 0.00 -> 4.58 mm
- net Net-(D9-A): track 0.00 -> 4.58 mm
- net Net-(D4-A): track 0.00 -> 4.58 mm
- net Net-(D14-A): track 0.00 -> 4.58 mm
- net Net-(D13-A): track 0.00 -> 4.58 mm
- net Net-(D12-A): track 0.00 -> 4.58 mm
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Other:
- board outline added: 78.2 x 122.4 mm

Commit message: case
Parts:
- SW1: value SW_SPST -> SW_SPDT; footprint Button_Switch_THT:SW_SPST_Omron_B3F-315x_Angled -> Personal:SS-12F23G5
- U1: footprint Seeed_Studio_XIAO_Series:XIAO-ESP32-S3-SMD_PAD -> xiao:XIAO-ESP32-S3-SMD_PAD
- moved SW1 68.1 mm to (139.1, 46.9)
- moved BT1 16.9 mm to (132.7, 41.4), turned to -90 degrees
- moved C1 13.1 mm to (140.9, 56.9), turned to -90 degrees
- moved U1 10.5 mm to (91.4, 59.4), turned to 90 degrees
- moved J1 5.51 mm to (104.9, 42.3)
- moved J2 5.51 mm to (100.5, 42.3)
- moved J3 5.17 mm to (99.4, 58.9)
- moved U2 3.49 mm to (132.8, 47.4)
- moved R1 2.42 mm to (125.0, 53.9)
- moved R2 2.42 mm to (114.9, 58.7)
- moved R3 2.42 mm to (114.9, 44.4)
- moved R4 2.42 mm to (125.0, 49.1)
- moved Q1 2.00 mm to (132.9, 57.4)
- turned S_*1 to 180 degrees
- turned S_+1 to 180 degrees
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Connections:
- SW1 pad 1: +BATT -> prot+
- SW1 pad 2: prot+ -> +BATT
Routing:
- net row_3: track 105.1 -> 0.00 mm
- net row_1: track 64.4 -> 0.00 mm
- net row_2: track 59.9 -> 0.00 mm
- net Net-(D16-A): track 14.1 -> 0.00 mm
- net Net-(D8-A): track 4.70 -> 0.00 mm
- net Net-(D7-A): track 4.58 -> 0.00 mm
- net Net-(D6-A): track 4.58 -> 0.00 mm
- net Net-(D3-A): track 4.58 -> 0.00 mm
- net Net-(D2-A): track 4.58 -> 0.00 mm
- net Net-(D5-A): track 4.58 -> 0.00 mm
- net Net-(D9-A): track 4.58 -> 0.00 mm
- net Net-(D4-A): track 4.58 -> 0.00 mm
- net Net-(D14-A): track 4.58 -> 0.00 mm
- net Net-(D13-A): track 4.58 -> 0.00 mm
- net Net-(D12-A): track 4.58 -> 0.00 mm
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Other:
- board size 78.2 x 122.4 mm -> 76.2 x 122 mm

Commit message: working on the case
Parts:
- moved C1 4.74 mm to (136.2, 56.3)
- moved D1 3.33 mm to (78.0, 65.4)
- moved Q1 2.91 mm to (130.0, 57.6)
- moved U1 1.81 mm to (91.4, 57.6)
- moved D4 1.43 mm to (130.4, 65.4)
Other:
- outline, holes or cut-outs redrawn
Changed lines of the file:
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@@
 	(footprint "ScottoKeebs_Components:Diode_DO-35"
 		(layer "F.Cu")
-		(at 131.8475 65.395)
+		(at 130.41875 65.395)
 		(descr "Diode, DO-35_SOD27 series, Axial, Horizontal, pin pitch=7.62mm, , length*diameter=4*2mm^2, , http://www.diodes.com/_files/packages/DO-35.pdf")
 		(tags "Diode DO-35_SOD27 series Axial Horizontal pin pitch 7.62mm  length 4mm diameter 2mm")
@@
 	(footprint "ScottoKeebs_Components:Diode_DO-35"
 		(layer "F.Cu")
-		(at 74.6975 65.395)
+		(at 78.03125 65.395)
 		(descr "Diode, DO-35_SOD27 series, Axial, Horizontal, pin pitch=7.62mm, , length*diameter=4*2mm^2, , http://www.diodes.com/_files/packages/DO-35.pdf")
 		(tags "Diode DO-35_SOD27 series Axial Horizontal pin pitch 7.62mm  length 4mm diameter 2mm")
@@
 	(footprint "FS8205A:SOP65P640X120-8N"
 		(layer "F.Cu")
-		(at 132.935 57.395 90)
+		(at 130.035 57.595 90)
 		(property "Reference" "Q1"
 			(at 4.7625 0 180)
@@
 	(footprint "xiao:XIAO-ESP32-S3-SMD_PAD"
 		(layer "F.Cu")
-		(at 91.435 59.405 90)
+		(at 91.435 57.595 90)
 		(property "Reference" "U1"
 			(at -2.2 -19.136 90)
@@
 	(footprint "Capacitor_THT:CP_Radial_Tantal_D4.5mm_P5.00mm"
 		(layer "F.Cu")
-		(at 140.935 56.895 -90)
+		(at 136.235 56.295 -90)
 		(descr "CP, Radial_Tantal series, Radial, pin pitch=5.00mm, diameter=4.5mm, height=10mm, Tantal Electrolytic Capacitor, http://cdn-reichelt.de/documents/datenblatt/B300/TANTAL-TB-Serie%23.pdf")
 		(tags "CP Radial_Tantal series Radial pin pitch 5.00mm diameter 4.5mm height 10mm Tantal Electrolytic Capacitor")
@@
 	)
 	(gr_rect
+		(start 69.935 63.395)
+		(end 73.935 65.395)
+		(stroke
+			(width 0.1)
+			(type default)
+		)
+		(fill no)
+		(layer "Eco1.User")
+	)
+	(gr_rect
+		(start 142.135 63.395)
+		(end 146.135 65.395)
+		(stroke
+			(width 0.1)
+			(type default)
+		)
+		(fill no)
+		(layer "Eco1.User")
+	)
+	(gr_circle
+		(center 127.085 122.545)
+		(end 129.735 122.545)
+		(stroke
+			(width 0.05)
+			(type default)
+		)
+		(fill no)
+		(layer "Edge.Cuts")
+	)
+	(gr_circle
+		(center 142.135 63.395)
+		(end 142.135 66.045)
+		(stroke
+			(width 0.05)
+			(type default)
+		)
+		(fill no)
+		(layer "Edge.Cuts")
+	)
+	(gr_circle
+		(center 88.985 103.495)
+		(end 91.635 103.495)
+		(stroke
+			(width 0.05)
+			(type default)
+		)
+		(fill no)
+		(layer "Edge.Cuts")
+	)
+	(gr_rect
 		(start 69.935 38.645)
 		(end 146.135 160.645)
 		(stroke
 			(width 0.05)
+			(type default)
+		)
+		(fill no)
+		(layer "Edge.Cuts")
+	)
+	(gr_circle
+		(center 127.085 84.445)
+		(end 129.735 84.445)
+		(stroke
+			(width 0.05)
+			(type default)
+		)
+		(fill no)
+		(layer "Edge.Cuts")
+	)
+	(gr_circle
+		(center 73.935 63.395)
+		(end 73.935 66.045)
+		(stroke
+			(width 0.05)

Commit message: case development
Parts:
- S_+1, S_enter1: footprint ScottoKeebs_Hotswap:Hotswap_MX_Plated_2.00u_90deg -> ScottoKeebs_Hotswap:Hotswap_MX_Plated_2.00u
- moved S_enter1 3.55 mm to (138.2, 144.8), turned to 90 degrees
- moved S_+1 3.46 mm to (139.5, 105.4), turned to 90 degrees

Commit message: art
Parts:
- U1: footprint xiao:XIAO-ESP32-S3-SMD_PAD -> Seeed_Studio_XIAO_Series:XIAO-ESP32-S3-SMD_PAD
- moved S_enter1 3.55 mm to (136.6, 141.6)
- moved S_+1 3.46 mm to (136.6, 103.5)
Routing:
- net col_4: track 0.00 -> 204.8 mm, vias 0 -> 1
- net pwr: track 0.00 -> 168.1 mm, vias 0 -> 2
- net GND: track 0.00 -> 166.3 mm, vias 0 -> 2
- net col_3: track 0.00 -> 138.2 mm, vias 0 -> 1
- net row_3: track 0.00 -> 132.1 mm
- net row_4: track 0.00 -> 130.9 mm
- net col_2: track 0.00 -> 122.7 mm, vias 0 -> 1
- net row_1: track 0.00 -> 113.6 mm, vias 0 -> 1
- net col_1: track 0.00 -> 113.5 mm, vias 0 -> 1
- net row_2: track 0.00 -> 91.1 mm
- net prot+: track 0.00 -> 67.9 mm
- net Net-(J1-Pin_2): track 0.00 -> 55.1 mm, vias 0 -> 1
- net Net-(J3-Pin_3): track 0.00 -> 44.5 mm, vias 0 -> 1
- net -BATT: track 0.00 -> 31.1 mm
- net Net-(U2-VCC): track 0.00 -> 22.6 mm, vias 0 -> 1
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
Commit message: fs8205
Parts:
- removed Q1: FS8205A, FS8205A:SOP65P640X120-8N
Routing:
- net Net-(U2-OD): track 15.3 -> 0.35 mm
- net -BATT: track 31.1 -> 24.0 mm
- net Net-(U2-OC): track 6.59 -> 0.00 mm
- net GND: track 166.3 -> 160.4 mm

Commit message: footprint and pcb final edits (pre silkscreen art)
Parts:
- added Q2: FS8205, FS8205:SOT95P280X145-6N, F.Cu at (129.4, 53.7)
- moved U2 3.43 mm to (129.4, 47.7)
- moved R2 1.73 mm to (113.3, 58.0)
- moved R3 1.73 mm to (113.3, 43.7)
- moved R1 1.73 mm to (123.4, 53.2)
- moved R4 1.73 mm to (123.4, 48.5)
- moved BT1 1.30 mm to (131.5, 41.7)
Routing:
- net GND: track 160.4 -> 171.5 mm, vias 2 -> 1
- net Net-(U2-OD): track 0.35 -> 9.42 mm
- net -BATT: track 24.0 -> 32.8 mm
- net col_2: track 122.7 -> 117.0 mm
- net Net-(J1-Pin_2): track 55.1 -> 60.8 mm
- net col_3: track 138.2 -> 132.6 mm
- net row_2: track 91.1 -> 96.7 mm
- net prot+: track 67.9 -> 72.6 mm
- net Net-(U2-OC): track 0.00 -> 4.15 mm
- net pwr: track 168.1 -> 164.3 mm
- net row_1: track 113.6 -> 117.1 mm
- net Net-(J3-Pin_3): track 44.5 -> 41.5 mm
- net Net-(U2-VCC): track 22.6 -> 20.2 mm, vias 1 -> 0
- net col_1: track 113.5 -> 115.2 mm
- net row_3: track 132.1 -> 133.3 mm
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