File: pcb/tactical-tenkey.kicad_pcb (KiCad board)
At the start: 2 copper layers, 76.2 x 122 mm, 46 parts, among them J1 io_side, J2 esp32_side, J3 OLED, Q2 FS8205, SW1 SW_SPDT, U1 XIAO-ESP32-S3-SMD, U2 DW01A

Commit message: final pcb touches
Parts:
- added G***: by sammothxc & kwarr, Personal:tactical_tenkey, B.Cu at (90.1, 46.8)
