File: pcb/tactical-tenkey.kicad_pcb (KiCad board)
At the start: 2 copper layers, 76.2 x 122 mm, 47 parts, among them J1 io_side, J2 esp32_side, J3 OLED, Q2 FS8205, SW1 SW_SPDT, U1 XIAO-ESP32-S3-SMD, U2 DW01A

Commit message: fix battery mgmt not working after switching off
Connections:
- R3 pad 1: prot+ -> +BATT
Routing:
- net +BATT: track 10.4 -> 30.3 mm
- net prot+: track 72.6 -> 61.5 mm
- net row_3: track 133.3 -> 133.9 mm
- net Net-(D10-A): track 19.7 -> 20.2 mm
- net Net-(D9-A): track 19.7 -> 20.2 mm
- net Net-(D2-A): track 19.7 -> 20.2 mm
- net Net-(D16-A): track 22.6 -> 23.1 mm
